Commit message: Added new URDF file with properly scaled and positioned links

File: urdf/garbagebot.urdf (robot description, URDF)
Before this commit: robot trashbot, 6 links, 5 joints
Links:
- removed link caster_back_left_link
- removed link caster_back_right_link
- removed link wheel_left_link
- removed link wheel_right_link
- added link wheel_back_left_link, mass 2.8498940e-02; collision cylinder length=0.018 radius=0.033; visual mesh filename=package://trashbot/meshes/trashbot_wheel_v1.stl scale=0.001 0.001 0.001
- added link wheel_back_right_link, mass 2.8498940e-02; collision cylinder length=0.018 radius=0.033; visual mesh filename=package://trashbot/meshes/trashbot_wheel_v1.stl scale=0.001 0.001 0.001
- added link wheel_front_left_link, mass 2.8498940e-02; collision cylinder length=0.018 radius=0.033; visual mesh filename=package://trashbot/meshes/trashbot_wheel_v1.stl scale=0.001 0.001 0.001
- added link wheel_front_right_link, mass 2.8498940e-02; collision cylinder length=0.018 radius=0.033; visual mesh filename=package://trashbot/meshes/trashbot_wheel_v1.stl scale=0.001 0.001 0.001
Joints:
- removed joint caster_back_left_joint
- removed joint caster_back_right_joint
- removed joint wheel_left_joint
- removed joint wheel_right_joint
- added joint wheel_back_left_joint: type fixed, parent base_link, child wheel_back_left_link, origin xyz=0.0 0.144 0.023 rpy=1.57 0 0, axis 0 0 1
- added joint wheel_back_right_joint: type fixed, parent base_link, child wheel_back_right_link, origin xyz=0.0 0.144 0.023 rpy=1.57 0 0, axis 0 0 1
- added joint wheel_front_left_joint: type fixed, parent base_link, child wheel_front_left_link, origin xyz=0.0 -0.144 0.023 rpy=-1.57 0 0, axis 0 0 1
- added joint wheel_front_right_joint: type fixed, parent base_link, child wheel_front_right_link, origin xyz=0.0 -0.144 0.023 rpy=-1.57 0 0, axis 0 0 1
